File: CAD/v.2/uStream.kicad_pcb_v2.kicad_pcb (KiCad board)
At the start: 2 copper layers, 150 x 75 mm, 70 parts, among them J1 Transformer_In, J2 Thermocouple junction, J3 MAX6675, J4 Mains+Heater, J5 Air Blower, Q1 BTA16-600B, Q2 STP55NF06, SW1 Heater Encoder, SW2 Control for Air blower, SW3 SW_SPST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

Commit message: schematic and pcb updated
Parts:
- added H5: MountingHole_3.2mm_M3, MountingHole:MountingHole_3.2mm_M3, F.Cu at (108.7, 64.4)
- added H6: MountingHole_3.2mm_M3, MountingHole:MountingHole_3.2mm_M3, F.Cu at (183.7, 64.4)
- added H7: MountingHole_3.2mm_M3, MountingHole:MountingHole_3.2mm_M3, F.Cu at (108.7, 95.4)
- added H8: MountingHole, MountingHole:MountingHole_3.2mm_M3, B.Cu at (183.7, 95.4)
- moved J4 15.2 mm to (195.8, 83.6), turned to -90 degrees
- moved U4 7.68 mm to (178.3, 76.6), turned to 180 degrees
- moved D3 0.36 mm to (183.6, 75.6)
Connections:
- J4 pad 1: /Hot -> /COLD
- J4 pad 4: /COLD -> /Hot
Routing:
- net Net-(U4-Pad1): track 83.6 -> 95.1 mm
- net GND: track 120.7 -> 130.6 mm, vias 16 -> 17
- net /4.7V: track 110.8 -> 107.9 mm
- net Net-(U4-Pad2): track 84.5 -> 86.7 mm
