File: CAD/v.2/uStream.kicad_sch_v.kicad_sch (KiCad schematic)
At the start: 72 parts, among them J1 Transformer_In, J2 Thermocouple junction, J3 MAX6675, J4 Mains+Heater, J5 Air Blower, Q1 BTA16-600B, Q2 STP55NF06, SW1 Heater Encoder, SW2 Control for Air blower, SW3 SW_SPST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

Commit message: schematic and pcb updated
Connections:
- net COLD: now also J4.1 (Pin_1); no longer J4.4 (Pin_4)
- net Hot: now also J4.4 (Pin_4); no longer J4.1 (Pin_1)
Other:
- moved on the sheet: J4
Changed lines of the file:
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@@
     (pin "2")
   )
-  (symbol (lib_id "Connector:Screw_Terminal_01x04") (at 273.05 27.94 0) (unit 1)
+  (symbol (lib_id "Connector:Screw_Terminal_01x04") (at 262.89 30.48 180) (unit 1)
     (in_bom yes) (on_board yes)
-    (property "Reference" "J4" (id 0) (at 275.59 20.32 0)
+    (property "Reference" "J4" (id 0) (at 260.35 38.1 0)
       (effects (font (size 1.27 1.27)) (justify left))
     )
-    (property "Value" "Mains+Heater" (id 1) (at 275.59 35.56 90)
+    (property "Value" "Mains+Heater" (id 1) (at 260.35 22.86 90)
       (effects (font (size 1.27 1.27)) (justify left))
     )
-    (property "Footprint" "TerminalBlock_Phoenix:TerminalBlock_Phoenix_MKDS-1,5-4-5.08_1x04_P5.08mm_Horizontal" (id 2) (at 273.05 27.94 0)
+    (property "Footprint" "TerminalBlock_Phoenix:TerminalBlock_Phoenix_MKDS-1,5-4-5.08_1x04_P5.08mm_Horizontal" (id 2) (at 262.89 30.48 0)
       (effects (font (size 1.27 1.27)) hide)
     )
-    (property "Datasheet" "~" (id 3) (at 273.05 27.94 0)
+    (property "Datasheet" "~" (id 3) (at 262.89 30.48 0)
       (effects (font (size 1.27 1.27)) hide)
     )
